File: fixture-friend/ff-core.kicad_sch (KiCad schematic)
At the start: 30 parts, among them J2 TSW-102-07-G-S, J7 USB_C_Receptacle_USB2.0_16P, U1 NCP1117ST33T3G, U2 W25Q128JVSIQ, U3 RP2040, X1 12MHz

Commit message: Add RP2040 debug interfaces
Connections:
- net GPIO14 is gone; now on net PROBE_SWDIO: U3.17 (GPIO14)
- net GPIO0: no longer names the net of U3.2 (GPIO0)
- net GPIO1: no longer names the net of U3.3 (GPIO1)
- net GPIO10 renamed SPI1_SCK
- net GPIO11 renamed SPI1_MOSI
- net GPIO12 renamed PROBE_SWCLK
- net GPIO13 renamed PROBE_SWDIO
- net GPIO4 renamed UART1_TX
- net GPIO5 renamed UART1_RX
- net GPIO8 renamed SPI1_MISO
- net GPIO9 renamed SPI1_CS_N
